File: pcb/TvMux.kicad_pcb (KiCad board)
At the start: 2 copper layers, 60 x 60 mm, 50 parts, among them J1 USB_B_Micro, J2 Conn_01x03_Female, J3 HDMI_A, Q1 BSS138, Q2 MMBT3904, Q3 MMBT3904, Q4 BSS138, Q5 BSS138, Q6 BSS138, SW1 PAIR, U1 CP2102N-Axx-xQFN24, U2 ESP32-WROOM-E, U3 AP7361C-33E

Commit message: PCB R1
Parts:
- moved C11 39.6 mm to (166.8, 106.8), turned to 180 degrees
- moved U3 36.2 mm to (169.5, 102.2)
- moved C9 33.0 mm to (163.8, 101.5), turned to 90 degrees
- moved C5 30.8 mm to (158.5, 71.5), turned to 180 degrees
- moved R11 26.2 mm to (158.5, 68.8)
- moved R2 21.5 mm to (126.8, 72.2), turned to -90 degrees
- moved Q4 19.9 mm to (141.2, 87.0), turned to 90 degrees
- moved R19 19.3 mm to (151.7, 101.5), turned to 180 degrees
- moved R8 18.6 mm to (146.2, 87.9), turned to 90 degrees
- moved Q5 17.9 mm to (151.1, 87.0), turned to 90 degrees
- moved R16 16.6 mm to (141.2, 91.0), turned to 180 degrees
- moved C8 16.5 mm to (145.2, 104.2), turned to -90 degrees
- moved R5 16.0 mm to (129.8, 72.2), turned to -90 degrees
- moved R4 14.5 mm to (120.5, 72.2), turned to -90 degrees
- moved R3 9.57 mm to (118.5, 72.2), turned to -90 degrees
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- renumbered C7 to C10, C10 to C11, C3 to C2, C11 to C3, C2 to C4, C9 to C5, C4 to C6, C5 to C7, C6 to C8, C8 to C9, D4 to D1, D6 to D2, D2 to D3, D3 to D4, D7 to D5, D5 to D6, D1 to D7, J3 to J1, J1 to J3, Q4 to Q1, Q5 to Q2, Q6 to Q3, Q3 to Q4, Q2 to Q5, Q1 to Q6, R15 to R1, R9 to R10, R8 to R12, R12 to R13, R6 to R14, R7 to R15, R5 to R16, R1 to R17, R2 to R18, R3 to R19, R18 to R2, R16 to R3, R19 to R4, R13 to R5, R14 to R6, R17 to R7, R4 to R8, R10 to R9, U2 to U1, U1 to U2
Connections:
- D1 pad 1: HDMI_DDC_SCL -> HDMI_HOT_PLUG_DETECT
- D1 pad 3: HDMI_DDC_SDA -> HDMI_5V
- D1 pad 4: HDMI_5V -> HDMI_DDC_SDA
- D1 pad 5: HDMI_CEC -> HDMI_DDC_SCL
- D1 pad 6: HDMI_HOT_PLUG_DETECT -> HDMI_CEC
Routing:
- net VBUS: track 0.00 -> 80.1 mm
- net GND: track 0.00 -> 77.0 mm, vias 0 -> 33
- net HDMI_CEC: track 0.00 -> 45.1 mm, vias 0 -> 4
- net DDC_SCL: track 0.00 -> 42.5 mm
- net HDMI_5V: track 0.00 -> 42.2 mm
- net DDC_SDA: track 0.00 -> 40.3 mm
- net RGB: track 0.00 -> 39.3 mm, vias 0 -> 2
- net U0_RXD: track 0.00 -> 37.2 mm, vias 0 -> 2
- net WII_PAIR: track 0.00 -> 37.1 mm, vias 0 -> 2
- net Net-(Q1-Pad2): track 0.00 -> 36.7 mm, vias 0 -> 2
- net 3V3: track 0.00 -> 36.1 mm, vias 0 -> 13
- net WII_TX: track 0.00 -> 35.8 mm
- net U0_TXD: track 0.00 -> 35.7 mm, vias 0 -> 2
- net CHIP_PU: track 0.00 -> 34.7 mm, vias 0 -> 2
- net WII_RX: track 0.00 -> 33.0 mm
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- added copper zone on In2.Cu, net 3V3
- added copper zone on In1.Cu, net GND
Other:
- copper layers 2 -> 4
- board text added: "TvMux - R1"

Commit message: esp idf wip
Parts:
- D7: renamed from D6; footprint Capacitor_SMD:C_0603_1608Metric -> LED_SMD:LED_0603_1608Metric
- renumbered C3 to C1, C8 to C10, C1 to C2, C2 to C3, C5 to C4, C4 to C5, C10 to C6, C6 to C7, C9 to C8, C7 to C9, D2 to D1, D1 to D2, D5 to D4, D4 to D5, D7 to D6, J2 to J1, J1 to J2, Q2 to Q1, Q3 to Q2, Q1 to Q3, Q6 to Q4, Q4 to Q5, Q5 to Q6, R6 to R10, R12 to R11, R8 to R12, R15 to R13, R16 to R14, R14 to R15, R19 to R16, R13 to R19, R11 to R2, R7 to R5, R2 to R6, R5 to R7, R9 to R8, R10 to R9
Other:
- board text added: "TvMux - R2"
- board text removed: "TvMux - R1"

Commit message: idf compiles
Parts:
- removed the D1 at (132.0, 80.5)
- removed the R2 at (158.5, 68.8)
- removed the R7 at (129.8, 72.2)
- removed the R8 at (158.5, 74.2)
- added J1: Conn_01x03_Male, Connector_PinHeader_2.54mm:PinHeader_1x03_P2.54mm_Vertical, F.Cu at (157.5, 64.6)
- added R1: 47K, Resistor_SMD:R_0603_1608Metric, F.Cu at (164.8, 64.4)
- added R3: 1K, Resistor_SMD:R_0603_1608Metric, F.Cu at (132.0, 68.6)
- R9: renamed from R10; value 10K -> 1M
- moved C5 26.7 mm to (132.0, 74.8), turned to 0 degrees
- moved C4 5.36 mm to (166.2, 67.4), turned to -90 degrees
- moved SW1 3.70 mm to (170.2, 67.5), turned to -90 degrees
- moved Q3 3.06 mm to (132.2, 71.2)
- renumbered C5 to C4, C4 to C5, D2 to D1, D3 to D2, D4 to D3, D5 to D4, D6 to D5, D7 to D6, J1 to J2, J2 to J3, J3 to J4, R11 to R10, R12 to R11, R13 to R12, R15 to R13, R16 to R15, R17 to R16, R18 to R17, R19 to R18, R1 to R2, R3 to R4, R4 to R5, R5 to R6, R6 to R7, R9 to R8
Connections:
- C5 pad 2: Net-(C5-Pad2) -> HDMI_HOT_PLUG_DETECT
- Q3 pad 1: 3V3 -> HDMI_HOT_PLUG_DETECT
- Q3 pad 2: Net-(Q1-Pad2) -> GND
- Q3 pad 3: Net-(D2-Pad1) -> Net-(Q3-Pad3)
- R9 pad 1: Net-(D2-Pad1) -> HDMI_HOT_PLUG_DETECT
- R9 pad 2: HDMI_5V -> GND
- U1 pad 30: unconnected-(U1-Pad30) -> Net-(R4-Pad1)
- U1 pad 31: Net-(C5-Pad2) -> Net-(U1-Pad31)
Routing:
- net Net-(Q1-Pad2): track 36.7 -> 0.00 mm, vias 2 -> 0
- net Net-(R4-Pad1): track 0.00 -> 30.4 mm, vias 0 -> 2
- net GND: track 77.0 -> 94.3 mm, vias 33 -> 31
- net Net-(D2-Pad1): track 12.1 -> 0.00 mm
- net HDMI_HOT_PLUG_DETECT: track 10.1 -> 21.3 mm
- net Net-(U1-Pad31): track 0.00 -> 10.7 mm
- net Net-(C5-Pad2): track 9.06 -> 0.00 mm
- net HDMI_5V: track 42.2 -> 34.4 mm
- net WII_PAIR: track 37.1 -> 42.4 mm
- net Net-(Q3-Pad3): track 0.00 -> 2.76 mm
- net Net-(J1-Pad3): track 0.00 -> 2.52 mm
- net 3V3: track 35.7 -> 34.0 mm, vias 13 -> 12
Other:
- board text added: "-PAIR"
- board text added: "-SETUP"
- board text added: "OFF"
- board text added: "ON"

Commit message: pcb updates
Parts:
- R12: renamed from R8; value 2K -> 1K
- moved R12 26.3 mm to (135.0, 89.2), turned to 90 degrees
- moved C4 2.18 mm to (165.4, 69.4)
- moved D3 1.41 mm to (137.4, 92.4)
- moved R2 0.60 mm to (165.4, 64.4)
- turned R3 to 180 degrees
- renumbered R2 to R1, R11 to R10, R12 to R11, R1 to R2, R9 to R8, R10 to R9
Connections:
- J1 pad 2: Net-(U1-Pad31) -> Net-(J1-Pin_2)
- R12 pad 1: Net-(R9-Pad1) -> Net-(U1-GPIO5)
- R3 pad 1: Net-(R4-Pad1) -> HOT_PLUG_DETECT
- U1 pad 16: unconnected-(U1-Pad16) -> HOT_PLUG_DETECT
- U1 pad 28: Net-(R9-Pad1) -> unconnected-(U1-GPIO17-Pad28)
- U1 pad 29: Net-(R9-Pad1) -> Net-(U1-GPIO5)
- U1 pad 30: Net-(R4-Pad1) -> Net-(J1-Pin_2)
- U1 pad 31: Net-(U1-Pad31) -> unconnected-(U1-GPIO19-Pad31)
Routing:
- net Net-(U1-GPIO5): track 0.00 -> 38.2 mm, vias 0 -> 2
- net Net-(R4-Pad1): track 30.4 -> 0.00 mm, vias 2 -> 0
- net HDMI_CEC: track 45.1 -> 15.3 mm, vias 4 -> 0
- net HOT_PLUG_DETECT: track 0.00 -> 20.3 mm
- net Net-(J1-Pin_2): track 0.00 -> 11.8 mm
- net Net-(U1-Pad31): track 10.7 -> 0.00 mm
- net Net-(R9-Pad1): track 8.08 -> 0.00 mm
- net HDMI_5V: track 34.4 -> 35.9 mm
- net GND: track 94.3 -> 93.2 mm
- net WII_PAIR: track 42.4 -> 43.2 mm
- net Net-(Q3-D): track 2.76 -> 3.44 mm
- net USB_P: track 29.1 -> 28.5 mm
