File: pcb/TvMux.kicad_sch (KiCad schematic)
At the start: 50 parts, among them J1 USB_B_Micro, J2 Conn_01x03_Female, J3 HDMI_A, Q1 BSS138, Q2 MMBT3904, Q3 MMBT3904, Q4 BSS138, Q5 BSS138, Q6 BSS138, SW1 PAIR, U1 CP2102N-Axx-xQFN24, U2 ESP32-WROOM-E, U3 AP7361C-33E

Commit message: PCB R1
Parts:
- renumbered C7 to C10, C10 to C11, C3 to C2, C11 to C3, C2 to C4, C9 to C5, C4 to C6, C5 to C7, C6 to C8, C8 to C9, D4 to D1, D6 to D2, D2 to D3, D3 to D4, D7 to D5, D5 to D6, D1 to D7, J3 to J1, J1 to J3, Q4 to Q1, Q5 to Q2, Q6 to Q3, Q3 to Q4, Q2 to Q5, Q1 to Q6, R15 to R1, R9 to R10, R8 to R12, R12 to R13, R6 to R14, R7 to R15, R5 to R16, R1 to R17, R2 to R18, R3 to R19, R18 to R2, R16 to R3, R19 to R4, R13 to R5, R14 to R6, R17 to R7, R4 to R8, R10 to R9, U2 to U1, U1 to U2
Connections:
- net HDMI_5V: now also D1.3 (K); no longer D1.4 (K)
- net HDMI_CEC: now also D1.6 (K); no longer D1.5 (K)
- net HDMI_DDC_SCL: now also D1.5 (K); no longer D1.1 (K)
- net HDMI_DDC_SDA: now also D1.4 (K); no longer D1.3 (K)
- net HDMI_HOT_PLUG_DETECT: now also D1.1 (K); no longer D1.6 (K)

Commit message: esp idf wip
Parts:
- D7: renamed from D6; footprint Capacitor_SMD:C_0603_1608Metric -> LED_SMD:LED_0603_1608Metric
- renumbered C3 to C1, C8 to C10, C1 to C2, C2 to C3, C5 to C4, C4 to C5, C10 to C6, C6 to C7, C9 to C8, C7 to C9, D2 to D1, D1 to D2, D5 to D4, D4 to D5, D7 to D6, J2 to J1, J1 to J2, Q2 to Q1, Q3 to Q2, Q1 to Q3, Q6 to Q4, Q4 to Q5, Q5 to Q6, R6 to R10, R12 to R11, R8 to R12, R15 to R13, R16 to R14, R14 to R15, R19 to R16, R13 to R19, R11 to R2, R7 to R5, R2 to R6, R5 to R7, R9 to R8, R10 to R9

Commit message: idf compiles
Parts:
- removed D1: 1N5819, Diode_SMD:D_SOD-323, symbol Diode:1N5819
- removed R2: 100K, Resistor_SMD:R_0603_1608Metric, symbol Device:R
- removed R7: 10K, Resistor_SMD:R_0603_1608Metric, symbol Device:R
- removed R8: 1M, Resistor_SMD:R_0603_1608Metric, symbol Device:R
- added J1: Conn_01x03_Male, Connector_PinHeader_2.54mm:PinHeader_1x03_P2.54mm_Vertical, symbol Connector:Conn_01x03_Male
- added R1: 47K, Resistor_SMD:R_0603_1608Metric, symbol Device:R
- added R3: 1K, Resistor_SMD:R_0603_1608Metric, symbol Device:R
- R9: renamed from R10; value 10K -> 1M
- renumbered C5 to C4, C4 to C5, D2 to D1, D3 to D2, D4 to D3, D5 to D4, D6 to D5, D7 to D6, J1 to J2, J2 to J3, J3 to J4, R11 to R10, R12 to R11, R13 to R12, R15 to R13, R16 to R15, R17 to R16, R18 to R17, R19 to R18, R1 to R2, R3 to R4, R4 to R5, R5 to R6, R6 to R7, R9 to R8
Connections:
- net 3V3: now also R1.1; no longer Q3.1 (G)
- net GND: now also Q3.2 (S), R9.2, J1.1 (Pin_1)
- net HDMI_5V: no longer R9.2
- net HDMI_HOT_PLUG_DETECT: now also C5.2, Q3.1 (G), R9.1
- net at Q3.3 (D): now also R3.2; no longer R9.1
- net at U1.30 (GPIO18): now also R3.1
- net at U1.31 (GPIO19): now also J1.2 (Pin_2); no longer C5.2
- new net: J1.3 (Pin_3), R1.2
- no-connect marks 36 -> 35
Other:
- moved on the sheet: C5, R9

Commit message: pcb updates
Parts:
- R12: renamed from R8; value 2K -> 1K
- renumbered R2 to R1, R11 to R10, R12 to R11, R1 to R2, R9 to R8, R10 to R9
Connections:
- net HOT_PLUG_DETECT: now reaches U1.16 (MTCK/GPIO13/ADC2_CH4)
- net HOT_PLUG_DETECT: now also R3.1
- net at R12.1, U1.29 (GPIO5): no longer U1.28 (GPIO17)
- net at U1.30 (GPIO18): now also J1.2 (Pin_2); no longer R3.1
- net at U1.31 (GPIO19): no longer J1.2 (Pin_2)
- no-connect marks 35 -> 36
Other:
- moved on the sheet: C4, C5, J1, Q3, R12, R2, R3, R8, SW1
